Commit message: effort, velocity values updated in cobot.urdf.xacro\ndynamics tag added in every joint

File: cobot_description/urdf/cobot.urdf.xacro (robot description, xacro)
@@ -6,9 +6,4 @@
   xmlns:xacro="http://www.ros.org/wiki/xacro">
   <link name="base_link"/>
-  <!-- <joint name="base_link__base" type="fixed">
-    <parent link="base_link"/>
-    <child link="base"/>
-    <origin xyz="0.0 0.0 0.0" rpy="0.0 0.0 0.0"/>
-  </joint> -->
   <joint name="base_link__base_stand" type="fixed">
     <parent link="base_link"/>
@@ -43,5 +38,6 @@
     <child link="base" />
     <axis xyz="0 0 1" />
-    <limit lower="-3.1416" upper="3.1416" effort="0" velocity="0" />
+    <limit lower="-3.1416" upper="3.1416" effort="5" velocity="5" />
+    <dynamics damping="10.0" friction="10.0"/>
   </joint>
   <link name="base">
@@ -72,5 +68,6 @@
     <child link="shoulder" />
     <axis xyz="0 1 0" />
-    <limit lower="-3.1416" upper="3.1416" effort="0" velocity="0" />
+    <limit lower="-3.1416" upper="3.1416" effort="5" velocity="5" />
+    <dynamics damping="10.0" friction="10.0"/>
   </joint>
   <link name="shoulder">
@@ -101,5 +98,6 @@
     <child link="elbow" />
     <axis xyz="0 1 0" />
-    <limit lower="-3.1416" upper="3.1416" effort="0" velocity="0" />
+    <limit lower="-3.1416" upper="3.1416" effort="5" velocity="5" />
+    <dynamics damping="10.0" friction="10.0"/>
   </joint>
   <link name="elbow">
@@ -130,5 +128,6 @@
     <child link="end_effector" />
     <axis xyz="0 1 0" />
-    <limit lower="-3.1416" upper="3.1416" effort="0" velocity="0" />
+    <limit lower="-3.1416" upper="3.1416" effort="5" velocity="5" />
+    <dynamics damping="10.0" friction="10.0"/>
   </joint>
   <link name="end_effector">
